File: Hardware/SuperGauge/SuperGauge.kicad_sch (KiCad schematic)
At the start: 30 parts, among them J101 USBC, J102 MainConn, J201 Tag Connect, U103 ATmega16U2, U104 TB6612FNG, U301 NCV1117ST50T3G, Y101 Crystal_GND24

Commit message: Fix DRC
Parts:
- removed U301: NCV1117ST50T3G, Package_TO_SOT_SMD:SOT-223, symbol Regulator_Linear:LM1117-5.0
- added D105: MBR0520LT, Diode_SMD:D_SOD-123, symbol Diode:MBR0520LT
- added U105: LM1117MP-5.0, Package_TO_SOT_SMD:SOT-223-3_TabPin2, symbol Regulator_Linear:LM1117MP-5.0
Connections:
- net +12V: now also U105.3 (VI)
- net +5V: now also D105.1 (K), U105.2 (VO); no longer J101.A4 (VBUS), J101.A9 (VBUS), J101.B4 (VBUS), J101.B9 (VBUS)
- net GND: now also U105.1 (GND)
- net L1: no longer names the net of U103.7 (PD1)
- net L2: no longer names the net of U103.8 (PD2)
- new net: D105.2 (A), J101.A4 (VBUS), J101.A9 (VBUS), J101.B4 (VBUS), J101.B9 (VBUS)
- no-connect marks 15 -> 17
Changed lines of the file:
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@@
   (junction (at 35.56 100.965) (diameter 0) (color 0 0 0 0)
   )
-  (junction (at 42.545 25.4) (diameter 0) (color 0 0 0 0)
-  )
   (junction (at 226.06 37.465) (diameter 0) (color 0 0 0 0)
   )
@@
   )
   (no_connect (at 93.98 130.81))
+  (no_connect (at 93.98 156.21))
   (no_connect (at 93.98 115.57))
   (no_connect (at 93.98 168.91))
@@
   (no_connect (at 93.98 161.29))
   (no_connect (at 93.98 148.59))
+  (no_connect (at 93.98 158.75))
   (wire (pts (xy 251.46 20.955) (xy 254 20.955))
     (stroke (width 0) (type default))
@@
     (stroke (width 0) (type default))
   )
-  (wire (pts (xy 108.585 156.21) (xy 93.98 156.21))
-    (stroke (width 0) (type default))
-  )
   (wire (pts (xy 57.15 33.02) (xy 57.15 34.29))
     (stroke (width 0) (type default))
@@
     (stroke (width 0) (type default))
   )
+  (wire (pts (xy 51.435 25.4) (xy 55.88 25.4))
+    (stroke (width 0) (type default))
+  )
   (wire (pts (xy 153.035 139.065) (xy 156.21 139.065))
     (stroke (width 0) (type default))
@@
     (stroke (width 0) (type default))
   )
-  (wire (pts (xy 108.585 158.75) (xy 93.98 158.75))
-    (stroke (width 0) (type default))
-  )
   (wire (pts (xy 262.255 27.305) (xy 262.255 28.575))
     (stroke (width 0) (type default))
@@
     (stroke (width 0) (type default))
   )
+  (wire (pts (xy 55.88 25.4) (xy 55.88 22.86))
+    (stroke (width 0) (type default))
+  )
   (wire (pts (xy 56.515 146.05) (xy 56.515 147.32))
     (stroke (width 0) (type default))
@@
     (stroke (width 0) (type default))
   )
-  (wire (pts (xy 41.275 25.4) (xy 42.545 25.4))
+  (wire (pts (xy 41.275 25.4) (xy 43.815 25.4))
     (stroke (width 0) (type default))
   )
@@
     (stroke (width 0) (type default))
   )
-  (wire (pts (xy 42.545 25.4) (xy 44.45 25.4))
-    (stroke (width 0) (type default))
-  )
   (wire (pts (xy 261.62 50.165) (xy 263.525 50.165))
     (stroke (width 0) (type default))
@@
   )
   (wire (pts (xy 26.67 100.965) (xy 26.67 102.87))
-    (stroke (width 0) (type default))
-  )
-  (wire (pts (xy 44.45 25.4) (xy 44.45 22.86))
     (stroke (width 0) (type default))
   )
@@
     (effects (font (size 1.27 1.27)) (justify left bottom))
   )
-  (label "L1" (at 108.585 156.21 180) (fields_autoplaced)
-    (effects (font (size 1.27 1.27)) (justify right bottom))
-  )
   (label "XTAL1" (at 48.895 120.65 0) (fields_autoplaced)
     (effects (font (size 1.27 1.27)) (justify left bottom))
-  )
-  (label "L2" (at 108.585 158.75 180) (fields_autoplaced)
-    (effects (font (size 1.27 1.27)) (justify right bottom))
   )
   (label "XTAL2" (at 26.67 86.995 270) (fields_autoplaced)
@@
     )
   )
+  (symbol (lib_id "Diode:MBR0520LT") (at 47.625 25.4 180) (unit 1)
+    (in_bom yes) (on_board yes) (dnp no)
+    (property "Reference" "D105" (at 41.91 20.32 0)
+      (effects (font (size 1.27 1.27)) (justify right))
+    )
+    (property "Value" "MBR0520LT" (at 41.91 22.86 0)
+      (effects (font (size 1.27 1.27)) (justify right))
+    )
+    (property "Footprint" "Diode_SMD:D_SOD-123" (at 47.625 20.955 0)
+      (effects (font (size 1.27 1.27)) hide)
+    )
+    (property "Datasheet" "http://www.onsemi.com/pub_link/Collateral/MBR0520LT1-D.PDF" (at 47.625 25.4 0)
+      (effects (font (size 1.27 1.27)) hide)
+    )
+    (property "LCSC#" "C165467" (at 47.625 25.4 90)
+      (effects (font (size 1.27 1.27)) hide)
+    )
+    (pin "1")
+    (pin "2")
+    (instances
+      (project "Buisness Card"
+        (path "/06c440f2-be37-4ee2-9b93-ecbe11945716"
+          (reference "D105") (unit 1)
+        )
+      )
+      (project "SuperGauge"
+        (path "/c760676c-d9ee-41ca-9f41-6b67ada36a22"
+          (reference "D105") (unit 1)
+        )
+      )
+    )
+  )
   (symbol (lib_id "power:+5V") (at 153.035 136.525 0) (unit 1)
     (in_bom yes) (on_board yes) (dnp no)
@@
         (path "/c760676c-d9ee-41ca-9f41-6b67ada36a22"
           (reference "#PWR0113") (unit 1)
+        )
+      )
+    )
+  )
+  (symbol (lib_id "Regulator_Linear:LM1117MP-5.0") (at 236.22 148.59 0) (unit 1)
+    (in_bom yes) (on_board yes) (dnp no) (fields_autoplaced)
+    (property "Reference" "U105" (at 236.22 142.24 0)
+      (effects (font (size 1.27 1.27)))
+    )
+    (property "Value" "LM1117MP-5.0" (at 236.22 144.78 0)
+      (effects (font (size 1.27 1.27)))
+    )
+    (property "Footprint" "Package_TO_SOT_SMD:SOT-223-3_TabPin2" (at 236.22 148.59 0)
+      (effects (font (size 1.27 1.27)) hide)
+    )
+    (property "Datasheet" "http://www.ti.com/lit/ds/symlink/lm1117.pdf" (at 236.22 148.59 0)
+      (effects (font (size 1.27 1.27)) hide)
+    )
+    (pin "1")
+    (pin "2")
+    (pin "3")
+    (instances
+      (project "SuperGauge"
+        (path "/c760676c-d9ee-41ca-9f41-6b67ada36a22"
+          (reference "U105") (unit 1)
         )
       )
@@
         (path "/e51b0d47-7e88-4bbf-adc2-21abe8ab62c1"
           (reference "#FLG0101") (unit 1)
-        )
-      )
-    )
-  )
-  (symbol (lib_id "power:+5V") (at 44.45 22.86 0) (unit 1)
-    (in_bom yes) (on_board yes) (dnp no)
-    (property "Reference" "#PWR0126" (at 44.45 26.67 0)
-      (effects (font (size 1.27 1.27)) hide)
-    )
-    (property "Value" "+5V" (at 44.45 19.05 0)
-      (effects (font (size 1.27 1.27)))
-    )
-    (property "Footprint" "" (at 44.45 22.86 0)
-      (effects (font (size 1.27 1.27)) hide)
-    )
-    (property "Datasheet" "" (at 44.45 22.86 0)
-      (effects (font (size 1.27 1.27)) hide)
-    )
-    (pin "1")
-    (instances
-      (project "SuperGauge"
-        (path "/c760676c-d9ee-41ca-9f41-6b67ada36a22"
-          (reference "#PWR0126") (unit 1)
-        )
-      )
-      (project "SuperButtonX1"
-        (path "/e51b0d47-7e88-4bbf-adc2-21abe8ab62c1"
-          (reference "#PWR0113") (unit 1)
         )
       )
@@
     )
   )
+  (symbol (lib_id "power:+5V") (at 55.88 22.86 0) (unit 1)
+    (in_bom yes) (on_board yes) (dnp no)
+    (property "Reference" "#PWR0126" (at 55.88 26.67 0)
+      (effects (font (size 1.27 1.27)) hide)
+    )
+    (property "Value" "+5V" (at 55.88 19.05 0)
+      (effects (font (size 1.27 1.27)))
+    )
+    (property "Footprint" "" (at 55.88 22.86 0)
+      (effects (font (size 1.27 1.27)) hide)
+    )
+    (property "Datasheet" "" (at 55.88 22.86 0)
+      (effects (font (size 1.27 1.27)) hide)
+    )
+    (pin "1")
+    (instances
+      (project "SuperGauge"
+        (path "/c760676c-d9ee-41ca-9f41-6b67ada36a22"
+          (reference "#PWR0126") (unit 1)
+        )
+      )
+      (project "SuperButtonX1"
+        (path "/e51b0d47-7e88-4bbf-adc2-21abe8ab62c1"
+          (reference "#PWR0113") (unit 1)
+        )
+      )
+    )
+  )
   (symbol (lib_id "power:+5V") (at 226.06 20.32 0) (unit 1)
     (in_bom yes) (on_board yes) (dnp no)
@@
         (path "/c760676c-d9ee-41ca-9f41-6b67ada36a22"
           (reference "#PWR0112") (unit 1)
-        )
-      )
-    )
-  )
-  (symbol (lib_id "Regulator_Linear:LM1117-5.0") (at 236.22 148.59 0) (unit 1)
-    (in_bom yes) (on_board yes) (dnp no)
-    (property "Reference" "U301" (at 238.76 154.94 0)
-      (effects (font (size 1.27 1.27)))
-    )
-    (property "Value" "NCV1117ST50T3G" (at 236.22 144.78 0)
-      (effects (font (size 1.27 1.27)))
-    )
-    (property "Footprint" "Package_TO_SOT_SMD:SOT-223" (at 236.22 148.59 0)
-      (effects (font (size 1.27 1.27)) hide)
-    )
-    (property "Datasheet" "http://www.ti.com/lit/ds/symlink/lm1117.pdf" (at 236.22 148.59 0)
-      (effects (font (size 1.27 1.27)) hide)
-    )
-    (pin "1")
-    (pin "2")
-    (pin "3")
-    (instances
-      (project "PendulumController"
-        (path "/56a36285-5fb6-4ce5-a89e-a1f5713a7d15/ddccc170-e5f2-4630-b82e-7e46ab8f3eab"
-          (reference "U301") (unit 1)
-        )
-      )
-      (project "SuperGauge"
-        (path "/c760676c-d9ee-41ca-9f41-6b67ada36a22"
-          (reference "U102") (unit 1)
         )
       )
@@
         )
       )
-    )
-  )
-  (symbol (lib_id "power:PWR_FLAG") (at 42.545 25.4 0) (unit 1)
-    (in_bom yes) (on_board yes) (dnp no) (fields_autoplaced)
-    (property "Reference" "#FLG0103" (at 42.545 23.495 0)
-      (effects (font (size 1.27 1.27)) hide)
-    )
-    (property "Value" "PWR_FLAG" (at 42.545 19.685 0)
-      (effects (font (size 1.27 1.27)) hide)
-    )
-    (property "Footprint" "" (at 42.545 25.4 0)
-      (effects (font (size 1.27 1.27)) hide)
-    )
-    (property "Datasheet" "~" (at 42.545 25.4 0)
-      (effects (font (size 1.27 1.27)) hide)
-    )
-    (pin "1")
-    (instances
-      (project "SuperGauge"
-        (path "/c760676c-d9ee-41ca-9f41-6b67ada36a22"
-          (reference "#FLG0103") (unit 1)
-        )
-      )
-      (project "SuperButtonX1"
-        (path "/e51b0d47-7e88-4bbf-adc2-21abe8ab62c1"
-          (reference "#FLG0102") (unit 1)
-        )
-      )
