File: Hardware/SuperGauge/SuperGauge.kicad_sch (KiCad schematic)
At the start: 31 parts, among them J101 USBC, J102 MainConn, J201 Tag Connect, U103 ATmega16U2, U104 TB6612FNG, U105 LM1117MP-5.0, Y101 Crystal_GND24

Commit message: RC time
Parts:
- U104: LCSC# (none) -> C141517
Other:
- title: (none) -> Super Gauge
Changed lines of the file:
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@@
 (kicad_sch (version 20230121) (generator eeschema)
   (paper "A4")
+  (title_block
+    (title "Super Gauge")
+    (date "${ISSUE}")
+    (rev "${FULL_REVISION}")
+  )
   (junction (at 251.46 20.955) (diameter 0) (color 0 0 0 0)
   )
@@
       (effects (font (size 1.27 1.27)) hide)
     )
+    (property "LCSC#" "C141517" (at 246.38 47.625 0)
+      (effects (font (size 1.27 1.27)) hide)
+    )

Commit message: Add cad, bump libs and more
Parts:
- J101: footprint Connector_USB:USB_C_Receptacle_XKB_U262-16XN-4BVC11 -> KenwoodFox:USB_C_Receptacle_XKB_U262-16XN-4BVC11_Full_Pads
Changed lines of the file:
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@@
       (effects (font (size 1.27 1.27)))
     )
-    (property "Footprint" "Connector_USB:USB_C_Receptacle_XKB_U262-16XN-4BVC11" (at 29.845 40.64 0)
+    (property "Footprint" "KenwoodFox:USB_C_Receptacle_XKB_U262-16XN-4BVC11_Full_Pads" (at 29.845 40.64 0)
       (effects (font (size 1.27 1.27)) hide)
     )
