File: Hardware/SuperGauge/SuperGauge.kicad_pcb (KiCad board)
At the start: 2 copper layers, 51 x 51 mm, 32 parts, among them J101 USBC, J102 MainConn, J103 Tag Connect, U103 ATmega16U2, U104 TB6612FNG, U105 LM1117MP-5.0, Y101 Crystal_GND24

Commit message: Add stencil marks
Other:
- board text added: "Stencil Cut size"
Changed lines of the file:
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@@
   (gr_circle (center -18.4755 4.925) (end -17.1155 4.925)
+    (stroke (width 0.15) (type default)) (fill none) (layer "Dwgs.User"))
+  (gr_rect (start -40 -40) (end 40 40)
     (stroke (width 0.15) (type default)) (fill none) (layer "Dwgs.User"))
   (gr_arc (start -25.4755 -1.975) (mid -18.062097 -18.061597) (end -1.9755 -25.475)
@@
     (effects (font (size 1.5 1.5) (thickness 0.25) bold) (justify left top))
   )
+  (gr_text "Stencil Cut size" (at 0 -41) (layer "Dwgs.User")
+    (effects (font (size 1 1) (thickness 0.15)) (justify bottom))
+  )
+  (dimension (type aligned) (layer "Dwgs.User")
+    (pts (xy 40 40) (xy 40 -40))
+    (height 3)
+    (gr_text "80.0000 mm" (at 41.85 0 90) (layer "Dwgs.User")
+      (effects (font (size 1 1) (thickness 0.15)))
+    )
+    (format (prefix "") (suffix "") (units 3) (units_format 1) (precision 4))
+    (style (thickness 0.15) (arrow_length 1.27) (text_position_mode 0) (extension_height 0.58642) (extension_offset 0.5) keep_text_aligned)
+  )
+  (dimension (type aligned) (layer "Dwgs.User")
+    (pts (xy 40 -40) (xy -40 -40))
+    (height 4)
+    (gr_text "80.0000 mm" (at 0 -45.15) (layer "Dwgs.User")
+      (effects (font (size 1 1) (thickness 0.15)))
+    )
+    (format (prefix "") (suffix "") (units 3) (units_format 1) (precision 4))
+    (style (thickness 0.15) (arrow_length 1.27) (text_position_mode 0) (extension_height 0.58642) (extension_offset 0.5) keep_text_aligned)
+  )
   (segment (start -5.7255 7.525) (end -4.2255 9.025) (width 0.5) (layer "F.Cu") (net 1))
