File: Hardware/SuperGauge/SuperGauge.kicad_pcb (KiCad board)
At the start: 2 copper layers, 51 x 51 mm, 32 parts, among them J101 USBC, J102 MainConn, J103 Tag Connect, U103 ATmega16U2, U104 TB6612FNG, U105 LM1117MP-5.0, Y101 Crystal_GND24

Commit message: Add cad, bump libs and more
Parts:
- J101: footprint Connector_USB:USB_C_Receptacle_XKB_U262-16XN-4BVC11 -> KenwoodFox:USB_C_Receptacle_XKB_U262-16XN-4BVC11_Full_Pads
Routing:
- net Net-(D105-A): track 19.3 -> 17.7 mm
- net GND: track 24.5 -> 25.3 mm
